Commit message: 20251020

File: urdf/cooperative_transportation_4ws.xacro (robot description, xacro)
@@ -20,5 +20,5 @@
 <xacro:property name="vehicle_inertia_coef" value="${sim_body_mass/fusion_vehicle_body_mass}" />
 <!-- 車輪 -->
-<xacro:property name="fusion_wheel_mass" value="${sim_wheel_mass}" />
+<xacro:property name="fusion_wheel_mass" value="20.0" />
 <xacro:property name="sim_wheel_mass" value="8.0" />
 <xacro:property name="wheel_inertia_coef" value="${sim_wheel_mass/fusion_wheel_mass}" />
@@ -31,19 +31,19 @@
 <xacro:property name="sliding_mechanism_mass" value="36.58325703660448" />
 <!-- 摺動機構 -->
-<xacro:property name="sliding_mechanism_damping" value="${(0.5*2*sqrt(100000*(carrier_inertia_coef/3 + linkage_point_mass)))/5.0}" /> <!-- ばね定数：1000~10000, 割合：50%-->
+<xacro:property name="sliding_mechanism_damping" value="${(0.5*2*sqrt(100000*(sim_carrier_mass/3 + linkage_point_mass)))/5.0}" /> <!-- ばね定数：1000~10000, 割合：50%-->
 <xacro:property name="sliding_mechanism_mu" value="0.3" />
-<xacro:property name="sliding_mechanism_friction" value="${sliding_mechanism_mu*gravitational_acceleration*(carrier_inertia_coef/3 + linkage_point_mass)}" />
+<xacro:property name="sliding_mechanism_friction" value="${sliding_mechanism_mu*gravitational_acceleration*(sim_carrier_mass/3 + linkage_point_mass)}" />
 <!-- ステアリング -->
-<xacro:property name="steering_damping" value="1.0" />
+<xacro:property name="steering_damping" value="5.0" />
 <xacro:property name="steering_mu" value="0.001" />
-<xacro:property name="steering_friction" value="${steering_mu * gravitational_acceleration * 0.25*(carrier_inertia_coef/3 + linkage_point_mass + sliding_mechanism_mass + sim_body_mass)}" />
+<xacro:property name="steering_friction" value="${steering_mu * gravitational_acceleration * 0.25*(sim_carrier_mass/3 + linkage_point_mass + sliding_mechanism_mass + sim_body_mass)}" />
 <!-- 摺動機構に乗っかている回転関節 -->
 <xacro:property name="rotational_joint_damping" value="0.02" />
 <xacro:property name="rotational_joint_mu" value="0.001" />
-<xacro:property name="rotational_joint_friction" value="${rotational_joint_mu * gravitational_acceleration * carrier_inertia_coef/3}" />
+<xacro:property name="rotational_joint_friction" value="${rotational_joint_mu * gravitational_acceleration * sim_carrier_mass/3}" />
 <!-- wheelの接地面の摩擦などを定義 -->
-<xacro:property name="wheel_surface_mu1" value="0.8"/>
-<xacro:property name="wheel_surface_mu2" value="0.6" />
-<xacro:property name="wheel_kp" value="2e4" />
+<xacro:property name="wheel_surface_mu1" value="0.7"/>
+<xacro:property name="wheel_surface_mu2" value="0.5" />
+<xacro:property name="wheel_kp" value="2e7" />
 <xacro:property name="wheel_kd" value="5.0" />
 <xacro:property name="wheel_minDepth" value="0.01" />
@@ -1155,5 +1155,5 @@
   <dynamics damping="${wheel_joint_damping}" friction="${wheel_joint_friction}"/>
   <axis xyz="0.0 1.0 -0.0"/>
-  <limit effort="100.0" velocity="200.0"/>
+  <limit effort="100.0" velocity="${1.0/0.153}"/>
 </joint>
 <joint name="v1_rear_right_steering" type="revolute">
@@ -1210,5 +1210,5 @@
   <dynamics damping="${wheel_joint_damping}" friction="${wheel_joint_friction}"/>
   <axis xyz="0.0 1.0 -0.0"/>
-  <limit effort="100.0" velocity="200.0"/>
+  <limit effort="100.0" velocity="${1.0/0.153}"/>
 </joint>
 <joint name="v1_front_left_wheel_rotation" type="continuous">
@@ -1218,5 +1218,5 @@
   <dynamics damping="${wheel_joint_damping}" friction="${wheel_joint_friction}"/>
   <axis xyz="0.0 1.0 -0.0"/>
-  <limit effort="100.0" velocity="200.0"/>
+  <limit effort="100.0" velocity="${1.0/0.153}"/>
 </joint>
 <joint name="v1_rear_left_wheel_rotation" type="continuous">
@@ -1226,5 +1226,5 @@
   <dynamics damping="${wheel_joint_damping}" friction="${wheel_joint_friction}"/>
   <axis xyz="0.0 1.0 -0.0"/>
-  <limit effort="100.0" velocity="200.0"/>
+  <limit effort="100.0" velocity="${1.0/0.153}"/>
 </joint>
 <!-- <joint name="linkage1_rotation" type="continuous">
@@ -1326,5 +1326,5 @@
   <dynamics damping="${wheel_joint_damping}" friction="${wheel_joint_friction}"/>
   <axis xyz="0.0 1.0 -0.0"/>
-  <limit effort="100.0" velocity="200.0"/>
+  <limit effort="100.0" velocity="${1.0/0.153}"/>
 </joint>
 <joint name="v2_rear_right_wheel_rotation" type="continuous">
@@ -1334,5 +1334,5 @@
   <dynamics damping="${wheel_joint_damping}" friction="${wheel_joint_friction}"/>
   <axis xyz="-0.0 1.0 -0.0"/>
-  <limit effort="100.0" velocity="200.0"/>
+  <limit effort="100.0" velocity="${1.0/0.153}"/>
 </joint>
 <joint name="v2_front_left_wheel_rotation" type="continuous">
@@ -1342,5 +1342,5 @@
   <dynamics damping="${wheel_joint_damping}" friction="${wheel_joint_friction}"/>
   <axis xyz="0.0 1.0 -0.0"/>
-  <limit effort="100.0" velocity="200.0"/>
+  <limit effort="100.0" velocity="${1.0/0.153}"/>
 </joint>
 <joint name="v2_rear_left_wheel_rotation" type="continuous">
@@ -1350,5 +1350,5 @@
   <dynamics damping="${wheel_joint_damping}" friction="${wheel_joint_friction}"/>
   <axis xyz="-0.0 1.0 -0.0"/>
-  <limit effort="100.0" velocity="200.0"/>
+  <limit effort="100.0" velocity="${1.0/0.153}"/>
 </joint>
 <joint name="v3_sliding_machine_to_body" type="fixed">
@@ -1405,5 +1405,5 @@
   <dynamics damping="${wheel_joint_damping}" friction="${wheel_joint_friction}"/>
   <axis xyz="0.0 1.0 -0.0"/>
-  <limit effort="100.0" velocity="200.0"/>
+  <limit effort="100.0" velocity="${1.0/0.153}"/>
 </joint>
 <joint name="v3_rear_right_wheel_rotation" type="continuous">
@@ -1413,5 +1413,5 @@
   <dynamics damping="${wheel_joint_damping}" friction="${wheel_joint_friction}"/>
   <axis xyz="0.0 1.0 -0.0"/>
-  <limit effort="100.0" velocity="200.0"/>
+  <limit effort="100.0" velocity="${1.0/0.153}"/>
 </joint>
 <joint name="v3_front_left_wheel_rotation" type="continuous">
@@ -1421,5 +1421,5 @@
   <dynamics damping="${wheel_joint_damping}" friction="${wheel_joint_friction}"/>
   <axis xyz="0.0 1.0 -0.0"/>
-  <limit effort="100.0" velocity="200.0"/>
+  <limit effort="100.0" velocity="${1.0/0.153}"/>
 </joint>
 <joint name="v3_rear_left_wheel_rotation" type="continuous">
@@ -1429,5 +1429,5 @@
   <dynamics damping="${wheel_joint_damping}" friction="${wheel_joint_friction}"/>
   <axis xyz="0.0 1.0 -0.0"/>
-  <limit effort="100.0" velocity="200.0"/>
+  <limit effort="100.0" velocity="${1.0/0.153}"/>
 </joint>
 <joint name="linkage_point_to_v1" type="prismatic">
