Commit message: 20251106

File: urdf/cooperative_transportation_4ws_flat.xacro (robot description, xacro)
@@ -49,7 +49,7 @@
 <xacro:property name="wheel_minDepth" value="0.01" />
 <xacro:property name="wheel_maxVel" value="0.5" />
-<xacro:include filename="$(find cooperative_transportation_4ws_description)/urdf/materials.xacro" />
-<xacro:include filename="$(find cooperative_transportation_4ws_description)/urdf/cooperative_transportation_4ws.trans" />
-<xacro:include filename="$(find cooperative_transportation_4ws_description)/urdf/cooperative_transportation_4ws.gazebo" />
+<xacro:include filename="$(find cooperative_transportation_4ws_backstepping)/urdf/materials.xacro" />
+<xacro:include filename="$(find cooperative_transportation_4ws_backstepping)/urdf/cooperative_transportation_4ws.trans" />
+<xacro:include filename="$(find cooperative_transportation_4ws_backstepping)/urdf/cooperative_transportation_4ws.gazebo" />
 <link name="base_link"/>
 <!-- <link name="carrier">
@@ -62,5 +62,5 @@
     <origin xyz="0 0 -0.6559999999999989" rpy="0 0 0"/>
     <geometry>
-      <mesh filename="package://cooperative_transportation_4ws_description/meshes/base_link.stl" scale="0.001 0.001 0.001"/>
+      <mesh filename="package://cooperative_transportation_4ws_backstepping/meshes/base_link.stl" scale="0.001 0.001 0.001"/>
     </geometry>
     <material name="yellow"/>
@@ -69,5 +69,5 @@
     <origin xyz="0 0 -0.6559999999999989" rpy="0 0 0"/>
     <geometry>
-      <mesh filename="package://cooperative_transportation_4ws_description/meshes/base_link.stl" scale="0.001 0.001 0.001"/>
+      <mesh filename="package://cooperative_transportation_4ws_backstepping/meshes/base_link.stl" scale="0.001 0.001 0.001"/>
     </geometry>
   </collision>
@@ -82,5 +82,5 @@
     <origin xyz="0 -0.057 -0.6559999999999989" rpy="0 0 0"/>
     <geometry>
-      <mesh filename="package://cooperative_transportation_4ws_newwheel_description/meshes/base_link.stl" scale="0.001 0.001 0.001"/>
+      <mesh filename="package://cooperative_transportation_4ws_backstepping/meshes/base_link.stl" scale="0.001 0.001 0.001"/>
     </geometry>
     <material name="_"/>
@@ -89,5 +89,5 @@
     <origin xyz="0 -0.057 -0.6559999999999989" rpy="0 0 0"/>
     <geometry>
-      <mesh filename="package://cooperative_transportation_4ws_newwheel_description/meshes/base_link.stl" scale="0.001 0.001 0.001"/>
+      <mesh filename="package://cooperative_transportation_4ws_backstepping/meshes/base_link.stl" scale="0.001 0.001 0.001"/>
     </geometry>
   </collision>
@@ -102,5 +102,5 @@
     <origin xyz="-1.150031 0.34248 -0.110215" rpy="0 0 0"/>
     <geometry>
-      <mesh filename="package://cooperative_transportation_4ws_description/meshes/new_wheel_2.stl" scale="0.001 0.001 0.001"/>
+      <mesh filename="package://cooperative_transportation_4ws_backstepping/meshes/new_wheel_2.stl" scale="0.001 0.001 0.001"/>
     </geometry>
     <material name="gray"/>
@@ -122,5 +122,5 @@
     <origin xyz="-1.15045 0.34248 -0.316" rpy="0 0 0"/>
     <geometry>
-      <mesh filename="package://cooperative_transportation_4ws_description/meshes/new_hinge_2.stl" scale="0.001 0.001 0.001"/>
+      <mesh filename="package://cooperative_transportation_4ws_backstepping/meshes/new_hinge_2.stl" scale="0.001 0.001 0.001"/>
     </geometry>
     <material name="_"/>
@@ -129,5 +129,5 @@
     <origin xyz="-1.15045 0.34248 -0.316" rpy="0 0 0"/>
     <geometry>
-      <mesh filename="package://cooperative_transportation_4ws_description/meshes/new_hinge_2.stl" scale="0.001 0.001 0.001"/>
+      <mesh filename="package://cooperative_transportation_4ws_backstepping/meshes/new_hinge_2.stl" scale="0.001 0.001 0.001"/>
     </geometry>
   </collision>
@@ -142,5 +142,5 @@
     <origin xyz="-2.05045 0.34248 -0.316" rpy="0 0 0"/>
     <geometry>
-      <mesh filename="package://cooperative_transportation_4ws_description/meshes/new_hinge_1.stl" scale="0.001 0.001 0.001"/>
+      <mesh filename="package://cooperative_transportation_4ws_backstepping/meshes/new_hinge_1.stl" scale="0.001 0.001 0.001"/>
     </geometry>
     <material name="_"/>
@@ -149,5 +149,5 @@
     <origin xyz="-2.05045 0.34248 -0.316" rpy="0 0 0"/>
     <geometry>
-      <mesh filename="package://cooperative_transportation_4ws_description/meshes/new_hinge_1.stl" scale="0.001 0.001 0.001"/>
+      <mesh filename="package://cooperative_transportation_4ws_backstepping/meshes/new_hinge_1.stl" scale="0.001 0.001 0.001"/>
     </geometry>
   </collision>
@@ -162,5 +162,5 @@
     <origin xyz="-2.05045 -0.45752 -0.316" rpy="0 0 0"/>
     <geometry>
-      <mesh filename="package://cooperative_transportation_4ws_description/meshes/new_hinge_3.stl" scale="0.001 0.001 0.001"/>
+      <mesh filename="package://cooperative_transportation_4ws_backstepping/meshes/new_hinge_3.stl" scale="0.001 0.001 0.001"/>
     </geometry>
     <material name="_"/>
@@ -169,5 +169,5 @@
     <origin xyz="-2.05045 -0.45752 -0.316" rpy="0 0 0"/>
     <geometry>
-      <mesh filename="package://cooperative_transportation_4ws_description/meshes/new_hinge_3.stl" scale="0.001 0.001 0.001"/>
+      <mesh filename="package://cooperative_transportation_4ws_backstepping/meshes/new_hinge_3.stl" scale="0.001 0.001 0.001"/>
     </geometry>
   </collision>
@@ -182,5 +182,5 @@
     <origin xyz="-1.15045 -0.45752 -0.316" rpy="0 0 0"/>
     <geometry>
-      <mesh filename="package://cooperative_transportation_4ws_description/meshes/new_hinge_4.stl" scale="0.001 0.001 0.001"/>
+      <mesh filename="package://cooperative_transportation_4ws_backstepping/meshes/new_hinge_4.stl" scale="0.001 0.001 0.001"/>
     </geometry>
     <material name="_"/>
@@ -189,5 +189,5 @@
     <origin xyz="-1.15045 -0.45752 -0.316" rpy="0 0 0"/>
     <geometry>
-      <mesh filename="package://cooperative_transportation_4ws_description/meshes/new_hinge_4.stl" scale="0.001 0.001 0.001"/>
+      <mesh filename="package://cooperative_transportation_4ws_backstepping/meshes/new_hinge_4.stl" scale="0.001 0.001 0.001"/>
     </geometry>
   </collision>
@@ -202,5 +202,5 @@
     <origin xyz="-1.60045 -0.05752 -0.421" rpy="0 0 0"/>
     <geometry>
-      <mesh filename="package://cooperative_transportation_4ws_description/meshes/v1_body_1.stl" scale="0.001 0.001 0.001"/>
+      <mesh filename="package://cooperative_transportation_4ws_backstepping/meshes/v1_body_1.stl" scale="0.001 0.001 0.001"/>
     </geometry>
     <material name="body_red"/>
@@ -209,5 +209,5 @@
     <origin xyz="-1.60045 -0.05752 -0.421" rpy="0 0 0"/>
     <geometry>
-      <mesh filename="package://cooperative_transportation_4ws_description/meshes/v1_body_1.stl" scale="0.001 0.001 0.001"/>
+      <mesh filename="package://cooperative_transportation_4ws_backstepping/meshes/v1_body_1.stl" scale="0.001 0.001 0.001"/>
     </geometry>
   </collision>
@@ -222,5 +222,5 @@
     <origin xyz="-1.15045 -0.05752 -0.336" rpy="0 0 0"/>
     <geometry>
-      <mesh filename="package://cooperative_transportation_4ws_description/meshes/v1_rear_1.stl" scale="0.001 0.001 0.001"/>
+      <mesh filename="package://cooperative_transportation_4ws_backstepping/meshes/v1_rear_1.stl" scale="0.001 0.001 0.001"/>
     </geometry>
     <material name="_"/>
@@ -229,5 +229,5 @@
     <origin xyz="-1.15045 -0.05752 -0.336" rpy="0 0 0"/>
     <geometry>
-      <mesh filename="package://cooperative_transportation_4ws_description/meshes/v1_rear_1.stl" scale="0.001 0.001 0.001"/>
+      <mesh filename="package://cooperative_transportation_4ws_backstepping/meshes/v1_rear_1.stl" scale="0.001 0.001 0.001"/>
     </geometry>
   </collision>
@@ -242,5 +242,5 @@
     <origin xyz="-2.05045 -0.05752 -0.336" rpy="0 0 0"/>
     <geometry>
-      <mesh filename="package://cooperative_transportation_4ws_description/meshes/v1_front_1.stl" scale="0.001 0.001 0.001"/>
+      <mesh filename="package://cooperative_transportation_4ws_backstepping/meshes/v1_front_1.stl" scale="0.001 0.001 0.001"/>
     </geometry>
     <material name="_"/>
@@ -249,5 +249,5 @@
     <origin xyz="-2.05045 -0.05752 -0.336" rpy="0 0 0"/>
     <geometry>
-      <mesh filename="package://cooperative_transportation_4ws_description/meshes/v1_front_1.stl" scale="0.001 0.001 0.001"/>
+      <mesh filename="package://cooperative_transportation_4ws_backstepping/meshes/v1_front_1.stl" scale="0.001 0.001 0.001"/>
     </geometry>
   </collision>
@@ -262,5 +262,5 @@
     <origin xyz="-2.050031 0.34248 -0.110215" rpy="0 0 0"/>
     <geometry>
-      <mesh filename="package://cooperative_transportation_4ws_description/meshes/new_wheel_1.stl" scale="0.001 0.001 0.001"/>
+      <mesh filename="package://cooperative_transportation_4ws_backstepping/meshes/new_wheel_1.stl" scale="0.001 0.001 0.001"/>
     </geometry>
     <material name="_"/>
@@ -304,5 +304,5 @@
     <origin xyz="-2.050031 -0.45752 -0.110215" rpy="0 0 0"/>
     <geometry>
-      <mesh filename="package://cooperative_transportation_4ws_description/meshes/new_wheel_3.stl" scale="0.001 0.001 0.001"/>
+      <mesh filename="package://cooperative_transportation_4ws_backstepping/meshes/new_wheel_3.stl" scale="0.001 0.001 0.001"/>
     </geometry>
     <material name="gray"/>
@@ -346,5 +346,5 @@
     <origin xyz="-1.150031 -0.45752 -0.110215" rpy="0 0 0"/>
     <geometry>
-      <mesh filename="package://cooperative_transportation_4ws_description/meshes/new_wheel_4.stl" scale="0.001 0.001 0.001"/>
+      <mesh filename="package://cooperative_transportation_4ws_backstepping/meshes/new_wheel_4.stl" scale="0.001 0.001 0.001"/>
     </geometry>
     <material name="gray"/>
@@ -388,5 +388,5 @@
     <origin xyz="-1.60045 -0.057547 -0.681" rpy="0 0 0"/>
     <geometry>
-      <mesh filename="package://cooperative_transportation_4ws_description/meshes/linkage_point1_1.stl" scale="0.001 0.001 0.001"/>
+      <mesh filename="package://cooperative_transportation_4ws_backstepping/meshes/linkage_point1_1.stl" scale="0.001 0.001 0.001"/>
     </geometry>
     <material name="_"/>
@@ -395,5 +395,5 @@
     <origin xyz="-1.60045 -0.057547 -0.681" rpy="0 0 0"/>
     <geometry>
-      <mesh filename="package://cooperative_transportation_4ws_description/meshes/linkage_point1_1.stl" scale="0.001 0.001 0.001"/>
+      <mesh filename="package://cooperative_transportation_4ws_backstepping/meshes/linkage_point1_1.stl" scale="0.001 0.001 0.001"/>
     </geometry>
   </collision>
@@ -408,5 +408,5 @@
     <origin xyz="0.799387 -1.443222 -0.681" rpy="0 0 0"/>
     <geometry>
-      <mesh filename="package://cooperative_transportation_4ws_description/meshes/linkage_point2_1.stl" scale="0.001 0.001 0.001"/>
+      <mesh filename="package://cooperative_transportation_4ws_backstepping/meshes/linkage_point2_1.stl" scale="0.001 0.001 0.001"/>
     </geometry>
     <material name="_"/>
@@ -415,5 +415,5 @@
     <origin xyz="0.799387 -1.443222 -0.681" rpy="0 0 0"/>
     <geometry>
-      <mesh filename="package://cooperative_transportation_4ws_description/meshes/linkage_point2_1.stl" scale="0.001 0.001 0.001"/>
+      <mesh filename="package://cooperative_transportation_4ws_backstepping/meshes/linkage_point2_1.stl" scale="0.001 0.001 0.001"/>
     </geometry>
   </collision>
@@ -428,5 +428,5 @@
     <origin xyz="0.8 1.329973 -0.681" rpy="0 0 0"/>
     <geometry>
-      <mesh filename="package://cooperative_transportation_4ws_description/meshes/linkage_point3_1.stl" scale="0.001 0.001 0.001"/>
+      <mesh filename="package://cooperative_transportation_4ws_backstepping/meshes/linkage_point3_1.stl" scale="0.001 0.001 0.001"/>
     </geometry>
     <material name="_"/>
@@ -435,5 +435,5 @@
     <origin xyz="0.8 1.329973 -0.681" rpy="0 0 0"/>
     <geometry>
-      <mesh filename="package://cooperative_transportation_4ws_description/meshes/linkage_point3_1.stl" scale="0.001 0.001 0.001"/>
+      <mesh filename="package://cooperative_transportation_4ws_backstepping/meshes/linkage_point3_1.stl" scale="0.001 0.001 0.001"/>
     </geometry>
   </collision>
@@ -448,5 +448,5 @@
     <origin xyz="0.799387 -1.443195 -0.421" rpy="0 0 0"/>
     <geometry>
-      <mesh filename="package://cooperative_transportation_4ws_description/meshes/v2body_1.stl" scale="0.001 0.001 0.001"/>
+      <mesh filename="package://cooperative_transportation_4ws_backstepping/meshes/v2body_1.stl" scale="0.001 0.001 0.001"/>
     </geometry>
     <material name="body_red"/>
@@ -455,5 +455,5 @@
     <origin xyz="0.799387 -1.443195 -0.421" rpy="0 0 0"/>
     <geometry>
-      <mesh filename="package://cooperative_transportation_4ws_description/meshes/v2body_1.stl" scale="0.001 0.001 0.001"/>
+      <mesh filename="package://cooperative_transportation_4ws_backstepping/meshes/v2body_1.stl" scale="0.001 0.001 0.001"/>
     </geometry>
   </collision>
@@ -468,5 +468,5 @@
     <origin xyz="1.249387 -1.443195 -0.336" rpy="0 0 0"/>
     <geometry>
-      <mesh filename="package://cooperative_transportation_4ws_description/meshes/v2_rear_1.stl" scale="0.001 0.001 0.001"/>
+      <mesh filename="package://cooperative_transportation_4ws_backstepping/meshes/v2_rear_1.stl" scale="0.001 0.001 0.001"/>
     </geometry>
     <material name="_"/>
@@ -475,5 +475,5 @@
     <origin xyz="1.249387 -1.443195 -0.336" rpy="0 0 0"/>
     <geometry>
-      <mesh filename="package://cooperative_transportation_4ws_description/meshes/v2_rear_1.stl" scale="0.001 0.001 0.001"/>
+      <mesh filename="package://cooperative_transportation_4ws_backstepping/meshes/v2_rear_1.stl" scale="0.001 0.001 0.001"/>
     </geometry>
   </collision>
@@ -488,5 +488,5 @@
     <origin xyz="0.349387 -1.443195 -0.336" rpy="0 0 0"/>
     <geometry>
-      <mesh filename="package://cooperative_transportation_4ws_description/meshes/v2_front_1.stl" scale="0.001 0.001 0.001"/>
+      <mesh filename="package://cooperative_transportation_4ws_backstepping/meshes/v2_front_1.stl" scale="0.001 0.001 0.001"/>
     </geometry>
     <material name="_"/>
@@ -495,5 +495,5 @@
     <origin xyz="0.349387 -1.443195 -0.336" rpy="0 0 0"/>
     <geometry>
-      <mesh filename="package://cooperative_transportation_4ws_description/meshes/v2_front_1.stl" scale="0.001 0.001 0.001"/>
+      <mesh filename="package://cooperative_transportation_4ws_backstepping/meshes/v2_front_1.stl" scale="0.001 0.001 0.001"/>
     </geometry>
   </collision>
@@ -508,5 +508,5 @@
     <origin xyz="0.349387 -1.043195 -0.316" rpy="0 0 0"/>
     <geometry>
-      <mesh filename="package://cooperative_transportation_4ws_description/meshes/new_hinge_11.stl" scale="0.001 0.001 0.001"/>
+      <mesh filename="package://cooperative_transportation_4ws_backstepping/meshes/new_hinge_11.stl" scale="0.001 0.001 0.001"/>
     </geometry>
     <material name="_"/>
@@ -515,5 +515,5 @@
     <origin xyz="0.349387 -1.043195 -0.316" rpy="0 0 0"/>
     <geometry>
-      <mesh filename="package://cooperative_transportation_4ws_description/meshes/new_hinge_11.stl" scale="0.001 0.001 0.001"/>
+      <mesh filename="package://cooperative_transportation_4ws_backstepping/meshes/new_hinge_11.stl" scale="0.001 0.001 0.001"/>
     </geometry>
   </collision>
@@ -528,5 +528,5 @@
     <origin xyz="1.249387 -1.043195 -0.316" rpy="0 0 0"/>
     <geometry>
-      <mesh filename="package://cooperative_transportation_4ws_description/meshes/new_hinge_12.stl" scale="0.001 0.001 0.001"/>
+      <mesh filename="package://cooperative_transportation_4ws_backstepping/meshes/new_hinge_12.stl" scale="0.001 0.001 0.001"/>
     </geometry>
     <material name="_"/>
@@ -535,5 +535,5 @@
     <origin xyz="1.249387 -1.043195 -0.316" rpy="0 0 0"/>
     <geometry>
-      <mesh filename="package://cooperative_transportation_4ws_description/meshes/new_hinge_12.stl" scale="0.001 0.001 0.001"/>
+      <mesh filename="package://cooperative_transportation_4ws_backstepping/meshes/new_hinge_12.stl" scale="0.001 0.001 0.001"/>
     </geometry>
   </collision>
@@ -548,5 +548,5 @@
     <origin xyz="0.349387 -1.843195 -0.316" rpy="0 0 0"/>
     <geometry>
-      <mesh filename="package://cooperative_transportation_4ws_description/meshes/new_hinge_10.stl" scale="0.001 0.001 0.001"/>
+      <mesh filename="package://cooperative_transportation_4ws_backstepping/meshes/new_hinge_10.stl" scale="0.001 0.001 0.001"/>
     </geometry>
     <material name="_"/>
@@ -555,5 +555,5 @@
     <origin xyz="0.349387 -1.843195 -0.316" rpy="0 0 0"/>
     <geometry>
-      <mesh filename="package://cooperative_transportation_4ws_description/meshes/new_hinge_10.stl" scale="0.001 0.001 0.001"/>
+      <mesh filename="package://cooperative_transportation_4ws_backstepping/meshes/new_hinge_10.stl" scale="0.001 0.001 0.001"/>
     </geometry>
   </collision>
@@ -568,5 +568,5 @@
     <origin xyz="1.249387 -1.843195 -0.316" rpy="0 0 0"/>
     <geometry>
-      <mesh filename="package://cooperative_transportation_4ws_description/meshes/new_hinge_7.stl" scale="0.001 0.001 0.001"/>
+      <mesh filename="package://cooperative_transportation_4ws_backstepping/meshes/new_hinge_7.stl" scale="0.001 0.001 0.001"/>
     </geometry>
     <material name="_"/>
@@ -575,5 +575,5 @@
     <origin xyz="1.249387 -1.843195 -0.316" rpy="0 0 0"/>
     <geometry>
-      <mesh filename="package://cooperative_transportation_4ws_description/meshes/new_hinge_7.stl" scale="0.001 0.001 0.001"/>
+      <mesh filename="package://cooperative_transportation_4ws_backstepping/meshes/new_hinge_7.stl" scale="0.001 0.001 0.001"/>
     </geometry>
   </collision>
@@ -588,5 +588,5 @@
     <origin xyz="0.349806 -1.043195 -0.110215" rpy="0 0 0"/>
     <geometry>
-      <mesh filename="package://cooperative_transportation_4ws_description/meshes/new_wheel_12.stl" scale="0.001 0.001 0.001"/>
+      <mesh filename="package://cooperative_transportation_4ws_backstepping/meshes/new_wheel_12.stl" scale="0.001 0.001 0.001"/>
     </geometry>
     <material name="_"/>
@@ -630,5 +630,5 @@
     <origin xyz="1.249806 -1.043195 -0.110215" rpy="0 0 0"/>
     <geometry>
-      <mesh filename="package://cooperative_transportation_4ws_description/meshes/new_wheel_11.stl" scale="0.001 0.001 0.001"/>
+      <mesh filename="package://cooperative_transportation_4ws_backstepping/meshes/new_wheel_11.stl" scale="0.001 0.001 0.001"/>
     </geometry>
     <material name="gray"/>
@@ -672,5 +672,5 @@
     <origin xyz="0.349806 -1.843195 -0.110215" rpy="0 0 0"/>
     <geometry>
-      <mesh filename="package://cooperative_transportation_4ws_description/meshes/new_wheel_7.stl" scale="0.001 0.001 0.001"/>
+      <mesh filename="package://cooperative_transportation_4ws_backstepping/meshes/new_wheel_7.stl" scale="0.001 0.001 0.001"/>
     </geometry>
     <material name="gray"/>
@@ -714,5 +714,5 @@
     <origin xyz="1.249806 -1.843195 -0.110215" rpy="0 0 0"/>
     <geometry>
-      <mesh filename="package://cooperative_transportation_4ws_description/meshes/new_wheel_10.stl" scale="0.001 0.001 0.001"/>
+      <mesh filename="package://cooperative_transportation_4ws_backstepping/meshes/new_wheel_10.stl" scale="0.001 0.001 0.001"/>
     </geometry>
     <material name="gray"/>
@@ -756,5 +756,5 @@
     <origin xyz="0.8 1.33 -0.421" rpy="0 0 0"/>
     <geometry>
-      <mesh filename="package://cooperative_transportation_4ws_description/meshes/v3_body_1.stl" scale="0.001 0.001 0.001"/>
+      <mesh filename="package://cooperative_transportation_4ws_backstepping/meshes/v3_body_1.stl" scale="0.001 0.001 0.001"/>
     </geometry>
     <material name="body_red"/>
@@ -763,5 +763,5 @@
     <origin xyz="0.8 1.33 -0.421" rpy="0 0 0"/>
     <geometry>
-      <mesh filename="package://cooperative_transportation_4ws_description/meshes/v3_body_1.stl" scale="0.001 0.001 0.001"/>
+      <mesh filename="package://cooperative_transportation_4ws_backstepping/meshes/v3_body_1.stl" scale="0.001 0.001 0.001"/>
     </geometry>
   </collision>
@@ -776,5 +776,5 @@
     <origin xyz="1.25 1.33 -0.336" rpy="0 0 0"/>
     <geometry>
-      <mesh filename="package://cooperative_transportation_4ws_description/meshes/v3_rear_1.stl" scale="0.001 0.001 0.001"/>
+      <mesh filename="package://cooperative_transportation_4ws_backstepping/meshes/v3_rear_1.stl" scale="0.001 0.001 0.001"/>
     </geometry>
     <material name="_"/>
@@ -783,5 +783,5 @@
     <origin xyz="1.25 1.33 -0.336" rpy="0 0 0"/>
     <geometry>
-      <mesh filename="package://cooperative_transportation_4ws_description/meshes/v3_rear_1.stl" scale="0.001 0.001 0.001"/>
+      <mesh filename="package://cooperative_transportation_4ws_backstepping/meshes/v3_rear_1.stl" scale="0.001 0.001 0.001"/>
     </geometry>
   </collision>
@@ -796,5 +796,5 @@
     <origin xyz="0.35 1.33 -0.336" rpy="0 0 0"/>
     <geometry>
-      <mesh filename="package://cooperative_transportation_4ws_description/meshes/v3_front_1.stl" scale="0.001 0.001 0.001"/>
+      <mesh filename="package://cooperative_transportation_4ws_backstepping/meshes/v3_front_1.stl" scale="0.001 0.001 0.001"/>
     </geometry>
     <material name="_"/>
@@ -803,5 +803,5 @@
     <origin xyz="0.35 1.33 -0.336" rpy="0 0 0"/>
     <geometry>
-      <mesh filename="package://cooperative_transportation_4ws_description/meshes/v3_front_1.stl" scale="0.001 0.001 0.001"/>
+      <mesh filename="package://cooperative_transportation_4ws_backstepping/meshes/v3_front_1.stl" scale="0.001 0.001 0.001"/>
     </geometry>
   </collision>
@@ -816,5 +816,5 @@
     <origin xyz="0.35 1.73 -0.316" rpy="0 0 0"/>
     <geometry>
-      <mesh filename="package://cooperative_transportation_4ws_description/meshes/new_hinge_5.stl" scale="0.001 0.001 0.001"/>
+      <mesh filename="package://cooperative_transportation_4ws_backstepping/meshes/new_hinge_5.stl" scale="0.001 0.001 0.001"/>
     </geometry>
     <material name="_"/>
@@ -823,5 +823,5 @@
     <origin xyz="0.35 1.73 -0.316" rpy="0 0 0"/>
     <geometry>
-      <mesh filename="package://cooperative_transportation_4ws_description/meshes/new_hinge_5.stl" scale="0.001 0.001 0.001"/>
+      <mesh filename="package://cooperative_transportation_4ws_backstepping/meshes/new_hinge_5.stl" scale="0.001 0.001 0.001"/>
     </geometry>
   </collision>
@@ -836,5 +836,5 @@
     <origin xyz="1.25 1.73 -0.316" rpy="0 0 0"/>
     <geometry>
-      <mesh filename="package://cooperative_transportation_4ws_description/meshes/new_hinge_6.stl" scale="0.001 0.001 0.001"/>
+      <mesh filename="package://cooperative_transportation_4ws_backstepping/meshes/new_hinge_6.stl" scale="0.001 0.001 0.001"/>
     </geometry>
     <material name="_"/>
@@ -843,5 +843,5 @@
     <origin xyz="1.25 1.73 -0.316" rpy="0 0 0"/>
     <geometry>
-      <mesh filename="package://cooperative_transportation_4ws_description/meshes/new_hinge_6.stl" scale="0.001 0.001 0.001"/>
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